File: Filter_PCB/Filter_PCB.kicad_pcb (KiCad board)
At the start: 2 copper layers, 43.8 x 15.2 mm, 25 parts, among them J1 Conn_01x06_Male, J2 Conn_Coaxial, J3 Conn_Coaxial, U1 MCP4728

Commit message: footprint replacement
Parts:
- D1, D2, D3, D4: footprint Diode_SMD:D_SOD-523 -> libs:D_SOD-523
- J1: footprint Connector_PinHeader_2.54mm:PinHeader_1x06_P2.54mm_Vertical -> libs:SMD_1x06_P2.54mm_Horizontal
- J2, J3: footprint Connector_Coaxial:SMA_Amphenol_132289_EdgeMount -> libs:SMA_generic_EdgeMount
- moved J1 5.99 mm to (128.0, 82.8), turned to 90 degrees
- moved J2 2.54 mm to (92.1, 90.2), turned to 0 degrees
- moved J3 2.54 mm to (135.9, 90.2), turned to 180 degrees
Other:
- net class RF1 added: clearance 0.4, trace_width 0.4, via_dia 0.8, via_drill 0.4
