File: Filter_PCB/Filter_PCB.sch (KiCad schematic (older format))
At the start: 25 parts, among them J1 Conn_01x06_Male, J2 Conn_Coaxial, J3 Conn_Coaxial, U1 MCP4728

Commit message: footprint replacement
Parts:
- D1, D2, D3, D4: footprint Diode_SMD:D_SOD-523 -> libs:D_SOD-523
- J1: footprint Connector_PinHeader_2.54mm:PinHeader_1x06_P2.54mm_Vertical -> libs:SMD_1x06_P2.54mm_Horizontal
- J2, J3: footprint Connector_Coaxial:SMA_Amphenol_132289_EdgeMount -> libs:SMA_generic_EdgeMount
Changed lines of the file:
@@
 EESchema Schematic File Version 4
+LIBS:Filter_PCB-cache
 EELAYER 30 0
 EELAYER END
@@
 F 0 "J2" H 2728 4538 50  0000 C CNN
 F 1 "Conn_Coaxial" H 2728 4447 50  0000 C CNN
-F 2 "Connector_Coaxial:SMA_Amphenol_132289_EdgeMount" H 2800 4300 50  0001 C CNN
+F 2 "libs:SMA_generic_EdgeMount" H 2800 4300 50  0001 C CNN
 F 3 " ~" H 2800 4300 50  0001 C CNN
 	1    2800 4300
@@
 F 0 "D1" H 3900 4516 50  0000 C CNN
 F 1 "D_Capacitance_ALT" H 3900 4425 50  0000 C CNN
-F 2 "Diode_SMD:D_SOD-523" H 3900 4300 50  0001 C CNN
+F 2 "libs:D_SOD-523" H 3900 4300 50  0001 C CNN
 F 3 "~" H 3900 4300 50  0001 C CNN
 	1    3900 4300
@@
 F 0 "D2" V 5154 4879 50  0000 L CNN
 F 1 "D_Capacitance_ALT" V 5245 4879 50  0000 L CNN
-F 2 "Diode_SMD:D_SOD-523" H 5200 4800 50  0001 C CNN
+F 2 "libs:D_SOD-523" H 5200 4800 50  0001 C CNN
 F 3 "~" H 5200 4800 50  0001 C CNN
 	1    5200 4800
@@
 F 0 "J3" H 9178 4538 50  0000 C CNN
 F 1 "Conn_Coaxial" H 9178 4447 50  0000 C CNN
-F 2 "Connector_Coaxial:SMA_Amphenol_132289_EdgeMount" H 9250 4300 50  0001 C CNN
+F 2 "libs:SMA_generic_EdgeMount" H 9250 4300 50  0001 C CNN
 F 3 " ~" H 9250 4300 50  0001 C CNN
 	1    9250 4300
@@
 F 0 "D4" H 8150 4516 50  0000 C CNN
 F 1 "D_Capacitance_ALT" H 8150 4425 50  0000 C CNN
-F 2 "Diode_SMD:D_SOD-523" H 8150 4300 50  0001 C CNN
+F 2 "libs:D_SOD-523" H 8150 4300 50  0001 C CNN
 F 3 "~" H 8150 4300 50  0001 C CNN
 	1    8150 4300
@@
 F 0 "D3" V 6804 4879 50  0000 L CNN
 F 1 "D_Capacitance_ALT" V 6895 4879 50  0000 L CNN
-F 2 "Diode_SMD:D_SOD-523" H 6850 4800 50  0001 C CNN
+F 2 "libs:D_SOD-523" H 6850 4800 50  0001 C CNN
 F 3 "~" H 6850 4800 50  0001 C CNN
 	1    6850 4800
@@
 F 0 "J1" H 1450 2600 50  0000 C CNN
 F 1 "Conn_01x06_Male" H 1500 2700 50  0000 C CNN
-F 2 "Connector_PinHeader_2.54mm:PinHeader_1x06_P2.54mm_Vertical" H 1950 2550 50  0001 C CNN
+F 2 "libs:SMD_1x06_P2.54mm_Horizontal" H 1950 2550 50  0001 C CNN
 F 3 "~" H 1950 2550 50  0001 C CNN
 	1    1950 2550
