File: Filter_PCB/Filter_PCB_4.kicad_pcb (KiCad board)
At the start: 2 copper layers, 43.8 x 15.2 mm, 25 parts, among them J1 Conn_01x06_Male, J2 Conn_Coaxial, J3 Conn_Coaxial, U1 MCP4728

Commit message: modifche AWR + PCB
Parts:
- moved L4 7.70 mm to (114.2, 89.6)
- moved D3 6.23 mm to (111.9, 93.0)
- moved C6 6.16 mm to (112.6, 91.1)
- moved C5 4.54 mm to (111.1, 89.6)
- moved L3 3.05 mm to (109.5, 91.1)
- moved C4 1.45 mm to (107.9, 89.6)
- moved D2 1.19 mm to (108.7, 93.0)
- moved R4 1.11 mm to (117.7, 86.6)
- moved L2 0.92 mm to (106.3, 91.1)
- moved R3 0.81 mm to (110.4, 87.1)
- moved C1 0.45 mm to (99.2, 90.2)
- moved D1 0.08 mm to (102.9, 90.2)
- moved J2 0.08 mm to (92.1, 90.2)
Routing:
- net /VB: track 11.7 -> 0.00 mm
- net /VA: track 9.23 -> 0.00 mm
- net Net-(C5-Pad1): track 5.32 -> 0.00 mm
- net Net-(C4-Pad1): track 5.32 -> 0.00 mm
- net Net-(C1-Pad1): track 4.29 -> 0.00 mm
- net Net-(C7-Pad1): track 4.29 -> 0.00 mm
- net Net-(D4-Pad2): track 3.47 -> 0.00 mm
- net Net-(D1-Pad2): track 3.47 -> 0.00 mm
- net Net-(C7-Pad2): track 3.47 -> 0.00 mm
- net Net-(C1-Pad2): track 3.47 -> 0.00 mm
- net Net-(C4-Pad2): track 1.60 -> 0.00 mm
- net Net-(C6-Pad2): track 1.60 -> 0.00 mm
- net Net-(C5-Pad2): track 1.60 -> 0.00 mm
- net GND: vias 3 -> 0
Other:
- copper layers 2 -> 4
Changed lines of the file:
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@@
-(kicad_pcb (version 20171130) (host pcbnew 5.1.4-e60b266~84~ubuntu16.04.1)
+(kicad_pcb (version 20171130) (host pcbnew "(5.1.5)-2")
   (general
     (thickness 1.6)
     (drawings 6)
-    (tracks 43)
+    (tracks 0)
     (zones 0)
     (modules 25)
@@
   (layers
     (0 F.Cu signal)
+    (1 In1.Cu power)
+    (2 In2.Cu power)
     (31 B.Cu signal)
     (32 B.Adhes user)
@@
     (35 F.Paste user)
     (36 B.SilkS user)
-    (37 F.SilkS user)
+    (37 F.SilkS user hide)
     (38 B.Mask user)
     (39 F.Mask user)
@@
     (via_min_size 0.4)
     (via_min_drill 0.3)
+    (user_via 0.5 0.3)
     (user_via 0.6 0.3)
     (uvia_size 0.3)
@@
     (solder_mask_min_width 0.25)
     (aux_axis_origin 0 0)
-    (visible_elements FFF9FF5F)
+    (visible_elements 7FFFFF5F)
     (pcbplotparams
       (layerselection 0x010fc_ffffffff)
@@
   )
   (module libs:D_SOD-523 (layer F.Cu)
-    (at 118.11 92.71 270)
+    (at 111.887 93.0275 270)
     (descr "http://www.diodes.com/datasheets/ap02001.pdf p.144")
     (tags "Diode SOD523")
@@
   )
   (module libs:D_SOD-523 (layer F.Cu)
-    (at 109.855 92.71 270)
+    (at 108.712 93.0275 270)
     (descr "http://www.diodes.com/datasheets/ap02001.pdf p.144")
     (tags "Diode SOD523")
@@
   )
   (module libs:D_SOD-523 (layer F.Cu)
-    (at 102.87 90.17)
+    (at 102.87 90.25)
     (descr "http://www.diodes.com/datasheets/ap02001.pdf p.144")
     (tags "Diode SOD523")
@@
   )
   (module libs:SMA_generic_EdgeMount (layer F.Cu)
-    (at 92.075 90.17)
+    (at 92.075 90.25)
     (fp_text reference J2 (at 2.25 -4.25) (layer F.SilkS)
       (effects (font (size 1 1) (thickness 0.15)))
@@
   )
   (module Capacitor_SMD:C_0603_1608Metric (layer F.Cu)
-    (at 118.745 90.17)
+    (at 112.649 91.059)
     (descr "Capacitor SMD 0603 (1608 Metric), square (rectangular) end terminal, IPC_7351 nominal, (Body size source: http://www.tortai-tech.com/upload/download/2011102023233369053.pdf), generated with kicad-footprint-generator")
     (tags capacitor)
@@
   )
   (module Resistor_SMD:R_0603_1608Metric (layer F.Cu)
-    (at 118.11 87.63 270)
+    (at 117.6655 86.614 270)
     (descr "Resistor SMD 0603 (1608 Metric), square (rectangular) end terminal, IPC_7351 nominal, (Body size source: http://www.tortai-tech.com/upload/download/2011102023233369053.pdf), generated with kicad-footprint-generator")
     (tags resistor)
@@
   )
   (module Resistor_SMD:R_0603_1608Metric (layer F.Cu)
-    (at 109.855 87.63 270)
+    (at 110.4265 87.0585 270)
     (descr "Resistor SMD 0603 (1608 Metric), square (rectangular) end terminal, IPC_7351 nominal, (Body size source: http://www.tortai-tech.com/upload/download/2011102023233369053.pdf), generated with kicad-footprint-generator")
     (tags resistor)
@@
   )
   (module Inductor_SMD:L_0603_1608Metric (layer F.Cu)
-    (at 121.92 90.17 180)
+    (at 114.2365 89.5985 180)
     (descr "Inductor SMD 0603 (1608 Metric), square (rectangular) end terminal, IPC_7351 nominal, (Body size source: http://www.tortai-tech.com/upload/download/2011102023233369053.pdf), generated with kicad-footprint-generator")
     (tags inductor)
@@
   )
   (module Inductor_SMD:L_0603_1608Metric (layer F.Cu)
-    (at 112.395 90.17)
+    (at 109.474 91.059)
     (descr "Inductor SMD 0603 (1608 Metric), square (rectangular) end terminal, IPC_7351 nominal, (Body size source: http://www.tortai-tech.com/upload/download/2011102023233369053.pdf), generated with kicad-footprint-generator")
     (tags inductor)
@@
   )
   (module Inductor_SMD:L_0603_1608Metric (layer F.Cu)
-    (at 106.045 90.17)
+    (at 106.299 91.059)
     (descr "Inductor SMD 0603 (1608 Metric), square (rectangular) end terminal, IPC_7351 nominal, (Body size source: http://www.tortai-tech.com/upload/download/2011102023233369053.pdf), generated with kicad-footprint-generator")
     (tags inductor)
@@
   )
   (module Capacitor_SMD:C_0603_1608Metric (layer F.Cu)
-    (at 115.57 90.17 180)
+    (at 111.0615 89.5985 180)
     (descr "Capacitor SMD 0603 (1608 Metric), square (rectangular) end terminal, IPC_7351 nominal, (Body size source: http://www.tortai-tech.com/upload/download/2011102023233369053.pdf), generated with kicad-footprint-generator")
     (tags capacitor)
@@
   )
   (module Capacitor_SMD:C_0603_1608Metric (layer F.Cu)
-    (at 109.22 90.17 180)
+    (at 107.8865 89.5985 180)
     (descr "Capacitor SMD 0603 (1608 Metric), square (rectangular) end terminal, IPC_7351 nominal, (Body size source: http://www.tortai-tech.com/upload/download/2011102023233369053.pdf), generated with kicad-footprint-generator")
     (tags capacitor)
@@
   )
   (module Capacitor_SMD:C_0603_1608Metric (layer F.Cu)
-    (at 99.695 90.17)
+    (at 99.25 90.25)
     (descr "Capacitor SMD 0603 (1608 Metric), square (rectangular) end terminal, IPC_7351 nominal, (Body size source: http://www.tortai-tech.com/upload/download/2011102023233369053.pdf), generated with kicad-footprint-generator")
     (tags capacitor)
@@
   (gr_line (start 92.075 95.885) (end 135.89 95.885) (layer Edge.Cuts) (width 0.05))
   (gr_line (start 92.075 80.645) (end 92.075 95.885) (layer Edge.Cuts) (width 0.05))
-  (segment (start 100.4825 90.17) (end 102.17 90.17) (width 0.635) (layer F.Cu) (net 1))
-  (segment (start 102.17 88.4825) (end 102.235 88.4175) (width 0.2032) (layer F.Cu) (net 1))
-  (segment (start 102.17 90.17) (end 102.17 88.4825) (width 0.2032) (layer F.Cu) (net 1))
-  (segment (start 94.615 90.17) (end 98.9075 90.17) (width 0.635) (layer F.Cu) (net 2))
-  (via (at 110.49 94.615) (size 0.8) (drill 0.4) (layers F.Cu B.Cu) (net 3))
-  (via (at 103.505 94.615) (size 0.8) (drill 0.4) (layers F.Cu B.Cu) (net 3))
-  (via (at 117.475 94.615) (size 0.8) (drill 0.4) (layers F.Cu B.Cu) (net 3))
-  (segment (start 106.8325 90.17) (end 108.4325 90.17) (width 0.635) (layer F.Cu) (net 6))
-  (segment (start 110.0075 88.57) (end 109.855 88.4175) (width 0.2032) (layer F.Cu) (net 7))
-  (segment (start 110.0075 90.17) (end 110.0075 88.57) (width 0.2032) (layer F.Cu) (net 7))
-  (segment (start 109.855 91.1225) (end 109.855 92.01) (width 0.635) (layer F.Cu) (net 7))
-  (segment (start 110.0075 90.17) (end 110.0075 90.97) (width 0.635) (layer F.Cu) (net 7))
-  (segment (start 110.0075 90.97) (end 109.855 91.1225) (width 0.635) (layer F.Cu) (net 7))
-  (segment (start 110.0075 90.17) (end 111.6075 90.17) (width 0.635) (layer F.Cu) (net 7))
-  (segment (start 113.1825 90.17) (end 114.7825 90.17) (width 0.635) (layer F.Cu) (net 8))
-  (segment (start 117.9575 90.17) (end 117.9575 90.97) (width 0.635) (layer F.Cu) (net 9))
-  (segment (start 118.11 91.1225) (end 118.11 92.01) (width 0.635) (layer F.Cu) (net 9))
-  (segment (start 117.9575 90.97) (end 118.11 91.1225) (width 0.635) (layer F.Cu) (net 9))
-  (segment (start 117.9575 90.17) (end 117.9575 89.37) (width 0.2032) (layer F.Cu) (net 9))
-  (segment (start 118.11 89.2175) (end 118.11 88.4175) (width 0.2032) (layer F.Cu) (net 9))
-  (segment (start 117.9575 89.37) (end 118.11 89.2175) (width 0.2032) (layer F.Cu) (net 9))
-  (segment (start 116.3575 90.17) (end 117.9575 90.17) (width 0.635) (layer F.Cu) (net 9))
-  (segment (start 119.5325 90.17) (end 121.1325 90.17) (width 0.635) (layer F.Cu) (net 10))
-  (segment (start 125.795 90.17) (end 125.795 89.2825) (width 0.2032) (layer F.Cu) (net 11))
-  (segment (start 125.73 89.2175) (end 125.73 88.4175) (width 0.2032) (layer F.Cu) (net 11))
-  (segment (start 125.795 89.2825) (end 125.73 89.2175) (width 0.2032) (layer F.Cu) (net 11))
-  (segment (start 125.795 90.17) (end 127.4825 90.17) (width 0.635) (layer F.Cu) (net 11))
-  (segment (start 129.0575 90.17) (end 133.35 90.17) (width 0.635) (layer F.Cu) (net 12))
-  (segment (start 103.57 91.8575) (end 103.505 91.9225) (width 0.2032) (layer F.Cu) (net 13))
-  (segment (start 103.57 90.17) (end 103.57 91.8575) (width 0.2032) (layer F.Cu) (net 13))
-  (segment (start 103.57 90.17) (end 105.2575 90.17) (width 0.635) (layer F.Cu) (net 13))
-  (segment (start 124.395 90.17) (end 124.395 91.0575) (width 0.2032) (layer F.Cu) (net 14))
-  (segment (start 124.46 91.1225) (end 124.46 91.9225) (width 0.2032) (layer F.Cu) (net 14))
-  (segment (start 124.395 91.0575) (end 124.46 91.1225) (width 0.2032) (layer F.Cu) (net 14))
-  (segment (start 122.7075 90.17) (end 124.395 90.17) (width 0.635) (layer F.Cu) (net 14))
-  (segment (start 102.235 86.8425) (end 102.235 83.185) (width 0.2032) (layer F.Cu) (net 19))
-  (segment (start 102.6 82.82) (end 107.655 82.82) (width 0.2032) (layer F.Cu) (net 19))
-  (segment (start 102.235 83.185) (end 102.6 82.82) (width 0.2032) (layer F.Cu) (net 19))
-  (segment (start 104.94 86.8425) (end 109.855 86.8425) (width 0.2032) (layer F.Cu) (net 20))
-  (segment (start 104.4575 83.5025) (end 104.4575 86.36) (width 0.2032) (layer F.Cu) (net 20))
-  (segment (start 107.655 83.32) (end 104.64 83.32) (width 0.2032) (layer F.Cu) (net 20))
-  (segment (start 104.4575 86.36) (end 104.94 86.8425) (width 0.2032) (layer F.Cu) (net 20))
-  (segment (start 104.64 83.32) (end 104.4575 83.5025) (width 0.2032) (layer F.Cu) (net 20))
   (zone (net 3) (net_name GND) (layer F.Cu) (hatch edge 0.508)
     (connect_pads thru_hole_only (clearance 0.254))
@@
       )
     )
-  )
-  (zone (net 0) (net_name "") (layer F.Cu) (hatch edge 0.508)
-    (connect_pads thru_hole_only (clearance 0.254))
-    (min_thickness 0.254)
-    (keepout (tracks allowed) (vias allowed) (copperpour not_allowed))
-    (fill (arc_segments 32) (thermal_gap 0.508) (thermal_bridge_width 0.508))
-    (polygon
-      (pts
-        (xy 139.065 92.71) (xy 88.9 92.71) (xy 88.9 87.63) (xy 139.065 87.63)
-      )
-    )

Commit message: RF layout
Parts:
- added C10: 4.7u, Capacitor_SMD:C_0603_1608Metric, B.Cu at (78.9, 47.5)
- added C8: 100n, Capacitor_SMD:C_0603_1608Metric, F.Cu at (88.8, 47.5)
- added C9: 100n, Capacitor_SMD:C_0603_1608Metric, B.Cu at (75.9, 47.5)
- added D5: BB202, libs:D_SOD-523, F.Cu at (81.8, 51.0)
- added D6: BB202, libs:D_SOD-523, F.Cu at (85.7, 47.5)
- added D7: BB202, libs:D_SOD-523, F.Cu at (88.0, 51.0)
- added R10: 100k, Resistor_SMD:R_0603_1608Metric, F.Cu at (87.2, 44.9)
- added R7: 100k, Resistor_SMD:R_0603_1608Metric, F.Cu at (81.0, 44.9)
- added R8: 100k, Resistor_SMD:R_0603_1608Metric, F.Cu at (84.1, 44.9)
- added R9: 100k, Resistor_SMD:R_0603_1608Metric, F.Cu at (84.9, 51.6)
- C1, C2, C3, C4, C5, C6, C7: value C -> 100n
- D1, D2, D3, D4: value D_Capacitance_ALT -> BB202
- J1: value Conn_01x06_Male -> Conn_Coaxial; footprint libs:SMD_1x06_P2.54mm_Horizontal -> libs:SMA_generic_EdgeMount
- J3: value Conn_Coaxial -> Conn_01x06_Male; footprint libs:SMA_generic_EdgeMount -> Connector_PinHeader_2.54mm:PinHeader_2x03_P2.54mm_Vertical_SMD; moved to B.Cu
- L1, L2, L3: value L -> L0; footprint Inductor_SMD:L_0603_1608Metric -> libs:Coilcraft_0603CS
- L4: value L -> 180R; moved to B.Cu
- R1, R2, R3, R4, R5, R6: value R -> 100k
- U1: moved to B.Cu
- moved J1 73.7 mm to (62.5, 49.0), turned to 0 degrees
- moved R5 66.7 mm to (77.9, 44.9), turned to 0 degrees
- moved J3 66.4 mm to (84.5, 48.1)
- moved D4 62.4 mm to (79.5, 47.5), turned to 0 degrees
- moved R4 59.8 mm to (74.8, 44.9), turned to 0 degrees
- moved R6 59.2 mm to (78.7, 51.6), turned to 180 degrees
- moved C7 58.2 mm to (87.2, 49.0), turned to 0 degrees
- moved D2 57.7 mm to (73.3, 47.5), turned to 0 degrees
- moved C2 57.6 mm to (70.2, 47.5), turned to 0 degrees
- moved R2 57.4 mm to (71.7, 44.9), turned to 0 degrees
- moved L1 56.9 mm to (71.8, 49.0), turned to 0 degrees
- moved C3 56.1 mm to (74.8, 49.0), turned to 0 degrees
- moved L4 55.9 mm to (77.4, 47.5), turned to 90 degrees
- moved D3 55.5 mm to (75.6, 51.0)
- moved R1 54.4 mm to (68.6, 44.9), turned to 0 degrees
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Connections:
- net /VA renamed /RF/V0
- net /VC renamed /RF/V2
- C1 pad 1: Net-(C1-Pad1) -> /RF/RFin
- C1 pad 2: Net-(C1-Pad2) -> /RF/inv0/Vd
- C2 pad 1: VDDA -> /RF/inv0/Vd
- C2 pad 2: GND -> /RF/res0/In
- C3 pad 1: VDD -> /RF/inv1/In
- C3 pad 2: GND -> /RF/inv1/Vd
- C4 pad 1: Net-(C4-Pad1) -> /RF/inv1/Vd
- C4 pad 2: Net-(C4-Pad2) -> /RF/res1/In
- C5 pad 1: Net-(C5-Pad1) -> /RF/inv2/In
- C5 pad 2: Net-(C5-Pad2) -> /RF/inv2/Vd
- C6 pad 1: Net-(C5-Pad1) -> /RF/inv2/Vd
- C6 pad 2: Net-(C6-Pad2) -> /RF/res2/In
- C7 pad 1: Net-(C7-Pad1) -> /RF/inv3/In
- C7 pad 2: Net-(C7-Pad2) -> /RF/inv3/Vd
- D1 pad 1: Net-(C1-Pad2) -> /RF/inv0/Vd
- D1 pad 2: Net-(D1-Pad2) -> GND
- D2 pad 1: Net-(C4-Pad1) -> /RF/res0/Vd+
- D2 pad 2: GND -> /RF/inv1/In
- D3 pad 1: Net-(C5-Pad1) -> /RF/inv1/Vd
- D4 pad 1: Net-(C7-Pad2) -> /RF/res1/Vd+
- D4 pad 2: Net-(D4-Pad2) -> /RF/inv2/In
- J1 pad 1: GND -> /RF/RFin
- J1 pad 2: /RDY -> GND
- J2 pad 1: Net-(C1-Pad1) -> /RF/RFout
- J3 pad 1: Net-(C7-Pad1) -> GND
- J3 pad 2: GND -> /logic/RDY
- L1 pad 1: VDDA -> /RF/res0/In
- L1 pad 2: VDD -> /RF/res0/Vd+
- L2 pad 1: Net-(D1-Pad2) -> /RF/res1/In
- L2 pad 2: Net-(C4-Pad2) -> /RF/res1/Vd+
- L3 pad 1: Net-(C4-Pad1) -> /RF/res2/In
- L3 pad 2: Net-(C5-Pad2) -> /RF/res2/Vd+
- L4 pad 1: Net-(D4-Pad2) -> VDDA
- L4 pad 2: Net-(C6-Pad2) -> VDD
- R1 pad 2: Net-(C1-Pad2) -> /RF/inv0/Vd
- R2 pad 1: Net-(D1-Pad2) -> /RF/V1
- R2 pad 2: GND -> /RF/res0/Vd+
- R3 pad 1: /VB -> /RF/inv1/In
- R3 pad 2: Net-(C4-Pad1) -> GND
- R4 pad 2: Net-(C5-Pad1) -> /RF/inv1/Vd
- R5 pad 1: Net-(D4-Pad2) -> /RF/V3
- R5 pad 2: GND -> /RF/res1/Vd+
- R6 pad 1: /VD -> /RF/inv2/In
- R6 pad 2: Net-(C7-Pad2) -> GND
- U1 pad 2: /SCL -> /logic/SCL
- U1 pad 3: /SDA -> /logic/SDA
- U1 pad 4: /~LDAC -> /logic/~LDAC
- U1 pad 5: /RDY -> /logic/RDY
- U1 pad 7: /VB -> /RF/V1
- U1 pad 9: /VD -> /RF/V3
Routing:
- net /RF/inv3/Vd: track 0.00 -> 5.43 mm
- net /RF/inv2/Vd: track 0.00 -> 5.43 mm
- net /RF/inv0/Vd: track 0.00 -> 5.43 mm
- net /RF/inv1/Vd: track 0.00 -> 5.43 mm
- net /RF/inv2/In: track 0.00 -> 4.41 mm
- net /RF/inv1/In: track 0.00 -> 4.41 mm
- net /RF/inv3/In: track 0.00 -> 4.41 mm
- net /RF/res2/Vd+: track 0.00 -> 4.15 mm
- net /RF/res1/Vd+: track 0.00 -> 4.15 mm
- net /RF/res0/Vd+: track 0.00 -> 4.15 mm
- net /RF/RFout: track 0.00 -> 3.19 mm
- net /RF/RFin: track 0.00 -> 3.19 mm
- net /RF/V1: track 0.00 -> 2.34 mm, vias 0 -> 2
- net /RF/V0: track 0.00 -> 2.34 mm, vias 0 -> 2
- net /RF/V2: track 0.00 -> 2.34 mm, vias 0 -> 2
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- added copper zone on In1.Cu, net GND
- added copper zone on In2.Cu, net GND
Other:
- board size 43.8 x 15.2 mm -> 32.4 x 8.9 mm
- net class Default: clearance 0.2 -> 0.15
- rule trace_clearance: 0.2 -> 0.15
- rule trace_min: 0.2 -> 0.127

Commit message: filter corrections
Parts:
- moved C10 3.72 mm to (76.7, 50.5), turned to 180 degrees
- moved L4 1.66 mm to (76.7, 49.0), turned to 0 degrees
- moved C9 0.80 mm to (76.7, 47.5), turned to 0 degrees
- moved U1 0.80 mm to (71.4, 48.5)
- moved J3 0.10 mm to (84.6, 48.1)
Routing:
- net /RF/V0: track 2.34 -> 30.6 mm
- net /RF/V1: track 2.34 -> 29.3 mm
- net /RF/V2: track 2.34 -> 27.0 mm
- net /RF/V3: track 1.17 -> 11.8 mm
- net GND: vias 67 -> 70
- net /logic/~LDAC: vias 1 -> 0

Commit message: PCB layout
Parts:
- moved C10 5.47 mm to (73.9, 45.8)
- moved U1 2.92 mm to (73.9, 50.0)
- moved C9 2.80 mm to (73.9, 47.4), turned to 180 degrees
- moved L4 2.45 mm to (76.2, 46.6), turned to 90 degrees
- moved J3 0.90 mm to (83.7, 48.1)
Connections:
- J3 pad 2: /logic/RDY -> VDD
- J3 pad 3: /logic/~LDAC -> /logic/SDA
- J3 pad 4: /logic/SDA -> /logic/SCL
- J3 pad 5: /logic/SCL -> /logic/~LDAC
- J3 pad 6: VDD -> /logic/RDY
Routing:
- net /logic/~LDAC: track 0.00 -> 11.8 mm
- net /logic/SDA: track 0.00 -> 11.8 mm
- net /RF/V2: track 27.0 -> 19.0 mm
- net VDD: track 0.00 -> 6.60 mm
- net /logic/SCL: track 0.00 -> 6.55 mm
- net /logic/RDY: track 0.00 -> 6.12 mm
- net /RF/V1: track 29.3 -> 23.8 mm
- net /RF/V3: track 11.8 -> 13.1 mm
- net GND: vias 70 -> 68
- added copper zone on B.Cu, net VDDA
Other:
- board text added: "GND"
- board text added: "L.Anastasio E.D'Amico"
- board text added: "RDY"
- board text added: "SCL"
- board text added: "SDA"
- board text added: "VDD"
- board text added: "~LDAC"
