File: Varactor_test_PCB/Varactor_test_PCB.kicad_pcb (KiCad board)
At the start: 2 copper layers, 14 x 7.6 mm, 6 parts, among them J1 Conn_Coaxial, J2 Conn_02x01

Commit message: jig
Parts:
- J2: moved to F.Cu
- moved R1 5.39 mm to (105.4, 70.9), turned to 90 degrees
- moved J2 0.76 mm to (110.7, 68.1)
- moved R2 0.13 mm to (110.7, 65.7)
Routing:
- net Net-(C1-Pad2): track 8.59 -> 2.82 mm
- net Net-(J2-Pad2): track 2.10 -> 6.06 mm
- net GND: vias 24 -> 38
Other:
- net class Default: clearance 0.2 -> 0
- rule trace_clearance: 0.2 -> 0
- board text added: "E. D'Amico L. Anastasio"
