File: PCB/Filter_PCB_4/Filter_PCB_4.sch (KiCad schematic (older format))
At the start: 0 parts

Commit message: PCB
Changed lines of the file:
@@
 S 4600 3700 550  500
 U 5E2D7233
-F0 "logic" 50
-F1 "logic.sch" 50
+F0 "DAC" 50
+F1 "DAC.sch" 50
 F2 "V_A" O R 5150 3800 50
 F3 "V_B" O R 5150 3900 50
