File: PCB/Filter_PCB_4/inverter.sch (KiCad schematic (older format))
At the start: 5 parts

Commit message: PCB updated
resistori 0603 sostituiti da resistori 0402
Parts:
- R1: footprint Resistor_SMD:R_0603_1608Metric -> Resistor_SMD:R_0402_1005Metric
Changed lines of the file:
@@
 $Descr A4 11693 8268
 encoding utf-8
-Sheet 3 10
+Sheet 9 10
 Title ""
 Date ""
@@
 AR Path="/5E2D6D86/5E30679B/5E2FB9D0" Ref="C5"  Part="1"
 AR Path="/5E2D6D86/5E3071CF/5E2FB9D0" Ref="C7"  Part="1"
+AR Path="/5E2F86AC/5E2FB9D0" Ref="C7"  Part="1"
+AR Path="/5E305E8C/5E2FB9D0" Ref="C7"  Part="1"
+AR Path="/5E30679B/5E2FB9D0" Ref="C7"  Part="1"
+AR Path="/5E3071CF/5E2FB9D0" Ref="C7"  Part="1"
 F 0 "C7" V 5002 3750 50  0000 C CNN
 F 1 "100n" V 4911 3750 50  0000 C CNN
@@
 AR Path="/5E2D6D86/5E30679B/5E2FB9D6" Ref="C6"  Part="1"
 AR Path="/5E2D6D86/5E3071CF/5E2FB9D6" Ref="C8"  Part="1"
+AR Path="/5E2F86AC/5E2FB9D6" Ref="C8"  Part="1"
+AR Path="/5E305E8C/5E2FB9D6" Ref="C8"  Part="1"
+AR Path="/5E30679B/5E2FB9D6" Ref="C8"  Part="1"
+AR Path="/5E3071CF/5E2FB9D6" Ref="C8"  Part="1"
 F 0 "C8" V 5802 3750 50  0000 C CNN
 F 1 "100n" V 5711 3750 50  0000 C CNN
@@
 AR Path="/5E2D6D86/5E30679B/5E2FB9DC" Ref="D10"  Part="1"
 AR Path="/5E2D6D86/5E3071CF/5E2FB9DC" Ref="D14"  Part="1"
+AR Path="/5E2F86AC/5E2FB9DC" Ref="D14"  Part="1"
+AR Path="/5E305E8C/5E2FB9DC" Ref="D14"  Part="1"
+AR Path="/5E30679B/5E2FB9DC" Ref="D14"  Part="1"
+AR Path="/5E3071CF/5E2FB9DC" Ref="D14"  Part="1"
 F 0 "D14" V 5254 4079 50  0000 L CNN
 F 1 "BB202" V 5345 4079 50  0000 L CNN
@@
 AR Path="/5E2D6D86/5E30679B/5E2FB9E2" Ref="#PWR012"  Part="1"
 AR Path="/5E2D6D86/5E3071CF/5E2FB9E2" Ref="#PWR016"  Part="1"
+AR Path="/5E2F86AC/5E2FB9E2" Ref="#PWR016"  Part="1"
+AR Path="/5E305E8C/5E2FB9E2" Ref="#PWR0103"  Part="1"
+AR Path="/5E30679B/5E2FB9E2" Ref="#PWR0107"  Part="1"
+AR Path="/5E3071CF/5E2FB9E2" Ref="#PWR0111"  Part="1"
 F 0 "#PWR016" H 5300 3900 50  0001 C CNN
 F 1 "GND" H 5305 3977 50  0000 C CNN
@@
 AR Path="/5E2D6D86/5E30679B/5E2FB9E8" Ref="R9"  Part="1"
 AR Path="/5E2D6D86/5E3071CF/5E2FB9E8" Ref="R13"  Part="1"
+AR Path="/5E2F86AC/5E2FB9E8" Ref="R13"  Part="1"
+AR Path="/5E305E8C/5E2FB9E8" Ref="R13"  Part="1"
+AR Path="/5E30679B/5E2FB9E8" Ref="R13"  Part="1"
+AR Path="/5E3071CF/5E2FB9E8" Ref="R13"  Part="1"
 F 0 "R13" H 5370 3346 50  0000 L CNN
 F 1 "100k" H 5370 3255 50  0000 L CNN
-F 2 "Resistor_SMD:R_0603_1608Metric" V 5230 3300 50  0001 C CNN
+F 2 "Resistor_SMD:R_0402_1005Metric" V 5230 3300 50  0001 C CNN
 F 3 "~" H 5300 3300 50  0001 C CNN
 	1    5300 3300
@@
 AR Path="/5E2D6D86/5E30679B/5E1858B3" Ref="D9"  Part="1"
 AR Path="/5E2D6D86/5E3071CF/5E1858B3" Ref="D13"  Part="1"
+AR Path="/5E2F86AC/5E1858B3" Ref="D13"  Part="1"
+AR Path="/5E305E8C/5E1858B3" Ref="D13"  Part="1"
+AR Path="/5E30679B/5E1858B3" Ref="D13"  Part="1"
+AR Path="/5E3071CF/5E1858B3" Ref="D13"  Part="1"
 F 0 "D13" V 4954 4079 50  0000 L CNN
 F 1 "BB202" V 5045 4079 50  0000 L CNN
@@
 AR Path="/5E2D6D86/5E30679B/5E1875FE" Ref="#PWR011"  Part="1"
 AR Path="/5E2D6D86/5E3071CF/5E1875FE" Ref="#PWR015"  Part="1"
+AR Path="/5E2F86AC/5E1875FE" Ref="#PWR015"  Part="1"
+AR Path="/5E305E8C/5E1875FE" Ref="#PWR0104"  Part="1"
+AR Path="/5E30679B/5E1875FE" Ref="#PWR0108"  Part="1"
+AR Path="/5E3071CF/5E1875FE" Ref="#PWR0112"  Part="1"
 F 0 "#PWR015" H 5000 3900 50  0001 C CNN
 F 1 "GND" H 5005 3977 50  0000 C CNN

Commit message: gerber
Parts:
- R1: footprint Resistor_SMD:R_0402_1005Metric -> Resistor_SMD:R_0603_1608Metric
Changed lines of the file:
@@
 AR Path="/5E2D6D86/5E30679B/5E2FB9D0" Ref="C5"  Part="1"
 AR Path="/5E2D6D86/5E3071CF/5E2FB9D0" Ref="C7"  Part="1"
-AR Path="/5E2F86AC/5E2FB9D0" Ref="C7"  Part="1"
-AR Path="/5E305E8C/5E2FB9D0" Ref="C7"  Part="1"
-AR Path="/5E30679B/5E2FB9D0" Ref="C7"  Part="1"
-AR Path="/5E3071CF/5E2FB9D0" Ref="C7"  Part="1"
 F 0 "C7" V 5002 3750 50  0000 C CNN
 F 1 "100n" V 4911 3750 50  0000 C CNN
@@
 AR Path="/5E2D6D86/5E30679B/5E2FB9D6" Ref="C6"  Part="1"
 AR Path="/5E2D6D86/5E3071CF/5E2FB9D6" Ref="C8"  Part="1"
-AR Path="/5E2F86AC/5E2FB9D6" Ref="C8"  Part="1"
-AR Path="/5E305E8C/5E2FB9D6" Ref="C8"  Part="1"
-AR Path="/5E30679B/5E2FB9D6" Ref="C8"  Part="1"
-AR Path="/5E3071CF/5E2FB9D6" Ref="C8"  Part="1"
 F 0 "C8" V 5802 3750 50  0000 C CNN
 F 1 "100n" V 5711 3750 50  0000 C CNN
@@
 AR Path="/5E2FB9DC" Ref="D?"  Part="1"
 AR Path="/5E2D6D86/5E2F86AC/5E2FB9DC" Ref="D2"  Part="1"
-AR Path="/5E2D6D86/5E305E8C/5E2FB9DC" Ref="D6"  Part="1"
-AR Path="/5E2D6D86/5E30679B/5E2FB9DC" Ref="D10"  Part="1"
-AR Path="/5E2D6D86/5E3071CF/5E2FB9DC" Ref="D14"  Part="1"
-AR Path="/5E2F86AC/5E2FB9DC" Ref="D14"  Part="1"
-AR Path="/5E305E8C/5E2FB9DC" Ref="D14"  Part="1"
-AR Path="/5E30679B/5E2FB9DC" Ref="D14"  Part="1"
-AR Path="/5E3071CF/5E2FB9DC" Ref="D14"  Part="1"
-F 0 "D14" V 5254 4079 50  0000 L CNN
+AR Path="/5E2D6D86/5E305E8C/5E2FB9DC" Ref="D4"  Part="1"
+AR Path="/5E2D6D86/5E30679B/5E2FB9DC" Ref="D6"  Part="1"
+AR Path="/5E2D6D86/5E3071CF/5E2FB9DC" Ref="D8"  Part="1"
+F 0 "D8" V 5254 4079 50  0000 L CNN
 F 1 "BB202" V 5345 4079 50  0000 L CNN
 F 2 "libs:D_SOD-523" H 5300 4000 50  0001 C CNN
@@
 AR Path="/5E2FB9E2" Ref="#PWR?"  Part="1"
 AR Path="/5E2D6D86/5E2F86AC/5E2FB9E2" Ref="#PWR04"  Part="1"
-AR Path="/5E2D6D86/5E305E8C/5E2FB9E2" Ref="#PWR08"  Part="1"
-AR Path="/5E2D6D86/5E30679B/5E2FB9E2" Ref="#PWR012"  Part="1"
-AR Path="/5E2D6D86/5E3071CF/5E2FB9E2" Ref="#PWR016"  Part="1"
-AR Path="/5E2F86AC/5E2FB9E2" Ref="#PWR016"  Part="1"
-AR Path="/5E305E8C/5E2FB9E2" Ref="#PWR0103"  Part="1"
-AR Path="/5E30679B/5E2FB9E2" Ref="#PWR0107"  Part="1"
-AR Path="/5E3071CF/5E2FB9E2" Ref="#PWR0111"  Part="1"
-F 0 "#PWR016" H 5300 3900 50  0001 C CNN
+AR Path="/5E2D6D86/5E305E8C/5E2FB9E2" Ref="#PWR07"  Part="1"
+AR Path="/5E2D6D86/5E30679B/5E2FB9E2" Ref="#PWR010"  Part="1"
+AR Path="/5E2D6D86/5E3071CF/5E2FB9E2" Ref="#PWR013"  Part="1"
+F 0 "#PWR013" H 5300 3900 50  0001 C CNN
 F 1 "GND" H 5305 3977 50  0000 C CNN
 F 2 "" H 5300 4150 50  0001 C CNN
@@
 AR Path="/5E2FB9E8" Ref="R?"  Part="1"
 AR Path="/5E2D6D86/5E2F86AC/5E2FB9E8" Ref="R1"  Part="1"
-AR Path="/5E2D6D86/5E305E8C/5E2FB9E8" Ref="R5"  Part="1"
-AR Path="/5E2D6D86/5E30679B/5E2FB9E8" Ref="R9"  Part="1"
-AR Path="/5E2D6D86/5E3071CF/5E2FB9E8" Ref="R13"  Part="1"
-AR Path="/5E2F86AC/5E2FB9E8" Ref="R13"  Part="1"
-AR Path="/5E305E8C/5E2FB9E8" Ref="R13"  Part="1"
-AR Path="/5E30679B/5E2FB9E8" Ref="R13"  Part="1"
-AR Path="/5E3071CF/5E2FB9E8" Ref="R13"  Part="1"
-F 0 "R13" H 5370 3346 50  0000 L CNN
+AR Path="/5E2D6D86/5E305E8C/5E2FB9E8" Ref="R4"  Part="1"
+AR Path="/5E2D6D86/5E30679B/5E2FB9E8" Ref="R7"  Part="1"
+AR Path="/5E2D6D86/5E3071CF/5E2FB9E8" Ref="R10"  Part="1"
+F 0 "R10" H 5370 3346 50  0000 L CNN
 F 1 "100k" H 5370 3255 50  0000 L CNN
-F 2 "Resistor_SMD:R_0402_1005Metric" V 5230 3300 50  0001 C CNN
+F 2 "Resistor_SMD:R_0603_1608Metric" V 5230 3300 50  0001 C CNN
 F 3 "~" H 5300 3300 50  0001 C CNN
 	1    5300 3300
@@
 AR Path="/5E1858B3" Ref="D?"  Part="1"
 AR Path="/5E2D6D86/5E2F86AC/5E1858B3" Ref="D1"  Part="1"
-AR Path="/5E2D6D86/5E305E8C/5E1858B3" Ref="D5"  Part="1"
-AR Path="/5E2D6D86/5E30679B/5E1858B3" Ref="D9"  Part="1"
-AR Path="/5E2D6D86/5E3071CF/5E1858B3" Ref="D13"  Part="1"
-AR Path="/5E2F86AC/5E1858B3" Ref="D13"  Part="1"
-AR Path="/5E305E8C/5E1858B3" Ref="D13"  Part="1"
-AR Path="/5E30679B/5E1858B3" Ref="D13"  Part="1"
-AR Path="/5E3071CF/5E1858B3" Ref="D13"  Part="1"
-F 0 "D13" V 4954 4079 50  0000 L CNN
+AR Path="/5E2D6D86/5E305E8C/5E1858B3" Ref="D3"  Part="1"
+AR Path="/5E2D6D86/5E30679B/5E1858B3" Ref="D5"  Part="1"
+AR Path="/5E2D6D86/5E3071CF/5E1858B3" Ref="D7"  Part="1"
+F 0 "D7" V 4954 4079 50  0000 L CNN
 F 1 "BB202" V 5045 4079 50  0000 L CNN
 F 2 "libs:D_SOD-523" H 5000 4000 50  0001 C CNN
@@
 AR Path="/5E1875FE" Ref="#PWR?"  Part="1"
 AR Path="/5E2D6D86/5E2F86AC/5E1875FE" Ref="#PWR03"  Part="1"
-AR Path="/5E2D6D86/5E305E8C/5E1875FE" Ref="#PWR07"  Part="1"
-AR Path="/5E2D6D86/5E30679B/5E1875FE" Ref="#PWR011"  Part="1"
-AR Path="/5E2D6D86/5E3071CF/5E1875FE" Ref="#PWR015"  Part="1"
-AR Path="/5E2F86AC/5E1875FE" Ref="#PWR015"  Part="1"
-AR Path="/5E305E8C/5E1875FE" Ref="#PWR0104"  Part="1"
-AR Path="/5E30679B/5E1875FE" Ref="#PWR0108"  Part="1"
-AR Path="/5E3071CF/5E1875FE" Ref="#PWR0112"  Part="1"
-F 0 "#PWR015" H 5000 3900 50  0001 C CNN
+AR Path="/5E2D6D86/5E305E8C/5E1875FE" Ref="#PWR06"  Part="1"
+AR Path="/5E2D6D86/5E30679B/5E1875FE" Ref="#PWR09"  Part="1"
+AR Path="/5E2D6D86/5E3071CF/5E1875FE" Ref="#PWR012"  Part="1"
+F 0 "#PWR012" H 5000 3900 50  0001 C CNN
 F 1 "GND" H 5005 3977 50  0000 C CNN
 F 2 "" H 5000 4150 50  0001 C CNN
