File: PCB/Filter_PCB_4_btob/Filter_PCB_4_btob.kicad_pcb (KiCad board)
At the start: 4 copper layers, 36.6 x 7.4 mm, 45 parts, among them J1 Conn_Coaxial, J2 Conn_Coaxial, J3 Conn_01x06_Male, U1 MCP4728

Commit message: gerber
Parts:
- added ?: , , F.Cu at (174.2, 98.5)
- moved R4 0.27 mm to (157.9, 103.3)
- moved C9 0.20 mm to (159.9, 98.9)
- moved L4 0.14 mm to (162.1, 99.6)
- moved R12 0.14 mm to (173.1, 103.3)
- moved R2 0.11 mm to (155.8, 103.3)
- moved R8 0.11 mm to (165.5, 103.3)
- moved R1 0.10 mm to (153.1, 98.4)
- moved R10 0.10 mm to (171.0, 103.3)
- moved R11 0.10 mm to (171.9, 98.4)
- moved R13 0.10 mm to (174.9, 98.4)
- moved R3 0.10 mm to (156.7, 98.4)
- moved R5 0.10 mm to (159.7, 98.4)
- moved R6 0.10 mm to (163.4, 103.3)
- moved R7 0.10 mm to (164.3, 98.4)
- moved R9 0.10 mm to (168.3, 98.4)
Routing:
- net /RF/V0: track 31.8 -> 29.3 mm
- net VDD: track 8.33 -> 6.06 mm
- net /RF/V3: track 12.8 -> 11.8 mm
- net /RF/V1: track 26.7 -> 26.0 mm
- net GND: vias 32 -> 34
Other:
- board text added: "1"
- board text added: "2"
- board text added: "3"
- board text added: "4"
- board text added: "5"
- board text added: "6"
